Commit message: Add Gazebo simulation support
Co-authored-by: Cursor <cursoragent@cursor.com>

File: el_a3_ros/el_a3_description/urdf/el_a3.urdf.xacro (robot description, xacro)
@@ -5,4 +5,7 @@
   <!-- Arguments -->
   <xacro:arg name="use_mock_hardware" default="false"/>
+  <xacro:arg name="use_gazebo" default="false"/>
+  <xacro:arg name="gazebo_ros2_control_params" default=""/>
+  <xacro:arg name="mesh_prefix" default="package://el_a3_description/meshes/"/>
   <xacro:arg name="can_interface" default="can0"/>
   <xacro:arg name="host_can_id" default="253"/>
@@ -11,4 +14,5 @@
   <xacro:property name="wrist_motor_type" value="$(arg wrist_motor_type)"/>
   <xacro:property name="wrist_effort" value="${5.5 if wrist_motor_type == 'RS05' else 6.0}"/>
+  <xacro:property name="mesh_prefix" value="$(arg mesh_prefix)"/>
   <!-- Include ros2_control -->
   <xacro:include filename="$(find el_a3_description)/urdf/el_a3_ros2_control.xacro"/>
@@ -38,5 +42,5 @@
       <origin xyz="-0.000643355 0 0.059" rpy="0 0 0"/>
       <geometry>
-        <mesh filename="package://el_a3_description/meshes/l1.stl"/>
+        <mesh filename="${mesh_prefix}l1.stl"/>
       </geometry>
       <material name="dark_brown"/>
@@ -45,5 +49,5 @@
       <origin xyz="-0.000643355 0 0.059" rpy="0 0 0"/>
       <geometry>
-        <mesh filename="package://el_a3_description/meshes/l1.stl"/>
+        <mesh filename="${mesh_prefix}l1.stl"/>
       </geometry>
     </collision>
@@ -60,5 +64,5 @@
       <origin xyz="-0.000642857 0 0.001" rpy="3.14159 0 0"/>
       <geometry>
-        <mesh filename="package://el_a3_description/meshes/l2.stl"/>
+        <mesh filename="${mesh_prefix}l2.stl"/>
       </geometry>
       <material name="orange"/>
@@ -67,5 +71,5 @@
       <origin xyz="-0.000642857 0 0.001" rpy="3.14159 0 0"/>
       <geometry>
-        <mesh filename="package://el_a3_description/meshes/l2.stl"/>
+        <mesh filename="${mesh_prefix}l2.stl"/>
       </geometry>
     </collision>
@@ -82,5 +86,5 @@
       <origin xyz="0.009 -0.07 0" rpy="-1.5708 0 0"/>
       <geometry>
-        <mesh filename="package://el_a3_description/meshes/l3.stl"/>
+        <mesh filename="${mesh_prefix}l3.stl"/>
       </geometry>
       <material name="dark_brown"/>
@@ -89,5 +93,5 @@
       <origin xyz="0.009 -0.07 0" rpy="-1.5708 0 0"/>
       <geometry>
-        <mesh filename="package://el_a3_description/meshes/l3.stl"/>
+        <mesh filename="${mesh_prefix}l3.stl"/>
       </geometry>
     </collision>
@@ -104,5 +108,5 @@
       <origin xyz="-0.181 -0.07 0" rpy="-1.5708 0 0"/>
       <geometry>
-        <mesh filename="package://el_a3_description/meshes/l4.stl"/>
+        <mesh filename="${mesh_prefix}l4.stl"/>
       </geometry>
       <material name="orange"/>
@@ -111,5 +115,5 @@
       <origin xyz="-0.181 -0.07 0" rpy="-1.5708 0 0"/>
       <geometry>
-        <mesh filename="package://el_a3_description/meshes/l4.stl"/>
+        <mesh filename="${mesh_prefix}l4.stl"/>
       </geometry>
     </collision>
@@ -126,5 +130,5 @@
       <origin xyz="0.004 0.134 0" rpy="1.5708 0 0"/>
       <geometry>
-        <mesh filename="package://el_a3_description/meshes/l5.stl"/>
+        <mesh filename="${mesh_prefix}l5.stl"/>
       </geometry>
       <material name="dark_brown"/>
@@ -133,5 +137,5 @@
       <origin xyz="0.004 0.134 0" rpy="1.5708 0 0"/>
       <geometry>
-        <mesh filename="package://el_a3_description/meshes/l5.stl"/>
+        <mesh filename="${mesh_prefix}l5.stl"/>
       </geometry>
     </collision>
@@ -148,5 +152,5 @@
       <origin xyz="0.0532 0 0.173" rpy="3.14159 0 0"/>
       <geometry>
-        <mesh filename="package://el_a3_description/meshes/l6.stl"/>
+        <mesh filename="${mesh_prefix}l6.stl"/>
       </geometry>
       <material name="orange"/>
@@ -155,5 +159,5 @@
       <origin xyz="0.0532 0 0.173" rpy="3.14159 0 0"/>
       <geometry>
-        <mesh filename="package://el_a3_description/meshes/l6.stl"/>
+        <mesh filename="${mesh_prefix}l6.stl"/>
       </geometry>
     </collision>
@@ -171,12 +175,12 @@
       <origin xyz="0 0 -0.0755" rpy="3.14159 0 0"/>
       <geometry>
-        <mesh filename="package://el_a3_description/meshes/el05_l6.stl"/>
-      </geometry>
-      <material name="dark_brown"/>
-    </visual>
-    <collision>
-      <origin xyz="0 0 -0.0755" rpy="3.14159 0 0"/>
-      <geometry>
-        <mesh filename="package://el_a3_description/meshes/el05_l6.stl"/>
+        <mesh filename="${mesh_prefix}el05_l6.stl"/>
+      </geometry>
+      <material name="dark_brown"/>
+    </visual>
+    <collision>
+      <origin xyz="0 0 -0.0755" rpy="3.14159 0 0"/>
+      <geometry>
+        <mesh filename="${mesh_prefix}el05_l6.stl"/>
       </geometry>
     </collision>
@@ -185,12 +189,12 @@
       <origin xyz="0 0 -0.0755" rpy="3.14159 0 0"/>
       <geometry>
-        <mesh filename="package://el_a3_description/meshes/jaw.stl"/>
-      </geometry>
-      <material name="orange"/>
-    </visual>
-    <collision>
-      <origin xyz="0 0 -0.0755" rpy="3.14159 0 0"/>
-      <geometry>
-        <mesh filename="package://el_a3_description/meshes/jaw.stl"/>
+        <mesh filename="${mesh_prefix}jaw.stl"/>
+      </geometry>
+      <material name="orange"/>
+    </visual>
+    <collision>
+      <origin xyz="0 0 -0.0755" rpy="3.14159 0 0"/>
+      <geometry>
+        <mesh filename="${mesh_prefix}jaw.stl"/>
       </geometry>
     </collision>
@@ -278,6 +282,14 @@
   <xacro:el_a3_ros2_control
     use_mock_hardware="$(arg use_mock_hardware)"
+    use_gazebo="$(arg use_gazebo)"
     can_interface="$(arg can_interface)"
     host_can_id="$(arg host_can_id)"
     wrist_motor_type="$(arg wrist_motor_type)"/>
+  <xacro:if value="$(arg use_gazebo)">
+    <gazebo>
+      <plugin name="gazebo_ros2_control" filename="libgazebo_ros2_control.so">
+        <parameters>$(arg gazebo_ros2_control_params)</parameters>
+      </plugin>
+    </gazebo>
+  </xacro:if>
 </robot>

File: el_a3_ros/el_a3_description/urdf/el_a3_ros2_control.xacro (robot description, xacro)
@@ -2,5 +2,5 @@
 <!-- EL-A3 ros2_control configuration -->
 <robot xmlns:xacro="http://www.ros.org/wiki/xacro">
-  <xacro:macro name="el_a3_ros2_control" params="use_mock_hardware can_interface host_can_id wrist_motor_type">
+  <xacro:macro name="el_a3_ros2_control" params="use_mock_hardware use_gazebo can_interface host_can_id wrist_motor_type">
     <!-- Wrist motor effort limits based on motor type -->
     <xacro:property name="wrist_effort_max" value="${5.5 if wrist_motor_type == 'RS05' else 6.0}"/>
@@ -8,69 +8,74 @@
     <ros2_control name="RsA3System" type="system">
       <hardware>
-        <xacro:if value="${use_mock_hardware}">
-          <plugin>mock_components/GenericSystem</plugin>
-          <param name="mock_sensor_commands">false</param>
+        <xacro:if value="${use_gazebo}">
+          <plugin>gazebo_ros2_control/GazeboSystem</plugin>
         </xacro:if>
-        <xacro:unless value="${use_mock_hardware}">
-          <plugin>el_a3_hardware/RsA3HardwareInterface</plugin>
-          <param name="can_interface">${can_interface}</param>
-          <param name="host_can_id">${host_can_id}</param>
-          <param name="position_kp">100.0</param>
-          <param name="position_kd">4.0</param>
-          <param name="velocity_limit">10.0</param>
-          <!-- S-curve trajectory planning parameters (source: s_curve_generator.cpp, not compiled yet) -->
-          <param name="s_curve_enabled">false</param>   <!-- Disabled: conflicts with MoveIt trajectory; enable after adding to CMakeLists.txt -->
-          <param name="max_velocity">3.0</param>        <!-- Max velocity limit rad/s -->
-          <param name="max_acceleration">15.0</param>   <!-- Max acceleration limit rad/s² -->
-          <param name="max_jerk">50.0</param>           <!-- Max jerk limit rad/s³ -->
-          <!-- Fallback smoothing filter parameters (used when S-curve is disabled) -->
-          <param name="smoothing_alpha">0.8</param>     <!-- Low-pass filter coefficient (0.8 = near-passthrough, teleop already smooths) -->
-          <!-- Gravity compensation feedforward parameters (100% gravity as feedforward torque, matching zero-torque mode) -->
-          <param name="gravity_feedforward_ratio">0.0</param>  <!-- Gravity feedforward disabled -->
-          <!-- Zero-torque mode parameters -->
-          <param name="zero_torque_kd">0.3</param>  <!-- Fixed Kd fallback (used when adaptive_kd disabled) -->
-          <!-- Velocity-adaptive Kd parameters (Lorentzian decay + EMA smoothing) -->
-          <param name="adaptive_kd_enabled">true</param>
-          <param name="zero_torque_kd_min">0.001</param>  <!-- Kd at high speed (smooth feel) -->
-          <param name="zero_torque_kd_max">0.15</param>   <!-- Kd at rest (stability) -->
-          <param name="kd_velocity_ref">1.0</param>        <!-- Reference velocity where Kd drops to midpoint (rad/s) -->
-          <param name="kd_smoothing_alpha">0.15</param>    <!-- EMA smoothing factor (smaller = smoother transitions) -->
-          <!-- Pinocchio dynamics model configuration -->
-          <param name="urdf_path">$(find el_a3_description)/urdf/el_a3.urdf</param>
-          <param name="use_pinocchio_gravity">true</param>  <!-- Enable full dynamics gravity compensation -->
-          <!-- Inertia parameter config file path (generated by inertia_calibration.py) -->
-          <param name="inertia_config_path">$(find el_a3_description)/config/inertia_params.yaml</param>
-          <!-- Inertia parameter scale factors (legacy method, kept for backward compatibility) -->
-          <param name="inertia_scale_L1_mass">1.0000</param>
-          <param name="inertia_scale_L2_mass">2.0000</param>
-          <param name="inertia_scale_L3_mass">0.6839</param>
-          <param name="inertia_scale_L4_mass">0.3500</param>
-          <param name="inertia_scale_L5_mass">1.0000</param>
-          <param name="inertia_scale_L6_mass">1.0000</param>
-          <!-- L1 joint - Base rotation around Z-axis, no gravity effect -->
-          <param name="gravity_comp_L1_sin">0.0</param>
-          <param name="gravity_comp_L1_cos">0.0</param>
-          <param name="gravity_comp_L1_offset">0.0</param>
-          <!-- L2 joint - Upper arm pitch, bears primary gravity load -->
-          <!-- τ = m*g*L*sin(θ), needs calibration based on actual measurements -->
-          <param name="gravity_comp_L2_sin">3.5</param>
-          <param name="gravity_comp_L2_cos">0.0</param>
-          <param name="gravity_comp_L2_offset">0.0</param>
-          <!-- L3 joint - Forearm pitch -->
-          <param name="gravity_comp_L3_sin">2.0</param>
-          <param name="gravity_comp_L3_cos">0.0</param>
-          <param name="gravity_comp_L3_offset">0.0</param>
-          <!-- L4 joint - Wrist Roll -->
-          <param name="gravity_comp_L4_sin">0.0</param>
-          <param name="gravity_comp_L4_cos">0.0</param>
-          <param name="gravity_comp_L4_offset">0.0</param>
-          <!-- L5 joint - Wrist Pitch -->
-          <param name="gravity_comp_L5_sin">0.3</param>
-          <param name="gravity_comp_L5_cos">0.0</param>
-          <param name="gravity_comp_L5_offset">0.0</param>
-          <!-- L6 joint - Wrist Yaw -->
-          <param name="gravity_comp_L6_sin">0.0</param>
-          <param name="gravity_comp_L6_cos">0.0</param>
-          <param name="gravity_comp_L6_offset">0.0</param>
+        <xacro:unless value="${use_gazebo}">
+          <xacro:if value="${use_mock_hardware}">
+            <plugin>mock_components/GenericSystem</plugin>
+            <param name="mock_sensor_commands">false</param>
+          </xacro:if>
+          <xacro:unless value="${use_mock_hardware}">
+            <plugin>el_a3_hardware/RsA3HardwareInterface</plugin>
+            <param name="can_interface">${can_interface}</param>
+            <param name="host_can_id">${host_can_id}</param>
+            <param name="position_kp">100.0</param>
+            <param name="position_kd">4.0</param>
+            <param name="velocity_limit">10.0</param>
+            <!-- S-curve trajectory planning parameters (source: s_curve_generator.cpp, not compiled yet) -->
+            <param name="s_curve_enabled">false</param>   <!-- Disabled: conflicts with MoveIt trajectory; enable after adding to CMakeLists.txt -->
+            <param name="max_velocity">3.0</param>        <!-- Max velocity limit rad/s -->
+            <param name="max_acceleration">15.0</param>   <!-- Max acceleration limit rad/s^2 -->
+            <param name="max_jerk">50.0</param>           <!-- Max jerk limit rad/s^3 -->
+            <!-- Fallback smoothing filter parameters (used when S-curve is disabled) -->
+            <param name="smoothing_alpha">0.8</param>     <!-- Low-pass filter coefficient (0.8 = near-passthrough, teleop already smooths) -->
+            <!-- Gravity compensation feedforward parameters (100% gravity as feedforward torque, matching zero-torque mode) -->
+            <param name="gravity_feedforward_ratio">0.0</param>  <!-- Gravity feedforward disabled -->
+            <!-- Zero-torque mode parameters -->
+            <param name="zero_torque_kd">0.3</param>  <!-- Fixed Kd fallback (used when adaptive_kd disabled) -->
+            <!-- Velocity-adaptive Kd parameters (Lorentzian decay + EMA smoothing) -->
+            <param name="adaptive_kd_enabled">true</param>
+            <param name="zero_torque_kd_min">0.001</param>  <!-- Kd at high speed (smooth feel) -->
+            <param name="zero_torque_kd_max">0.15</param>   <!-- Kd at rest (stability) -->
+            <param name="kd_velocity_ref">1.0</param>        <!-- Reference velocity where Kd drops to midpoint (rad/s) -->
+            <param name="kd_smoothing_alpha">0.15</param>    <!-- EMA smoothing factor (smaller = smoother transitions) -->
+            <!-- Pinocchio dynamics model configuration -->
+            <param name="urdf_path">$(find el_a3_description)/urdf/el_a3.urdf</param>
+            <param name="use_pinocchio_gravity">true</param>  <!-- Enable full dynamics gravity compensation -->
+            <!-- Inertia parameter config file path (generated by inertia_calibration.py) -->
+            <param name="inertia_config_path">$(find el_a3_description)/config/inertia_params.yaml</param>
+            <!-- Inertia parameter scale factors (legacy method, kept for backward compatibility) -->
+            <param name="inertia_scale_L1_mass">1.0000</param>
+            <param name="inertia_scale_L2_mass">2.0000</param>
+            <param name="inertia_scale_L3_mass">0.6839</param>
+            <param name="inertia_scale_L4_mass">0.3500</param>
+            <param name="inertia_scale_L5_mass">1.0000</param>
+            <param name="inertia_scale_L6_mass">1.0000</param>
+            <!-- L1 joint - Base rotation around Z-axis, no gravity effect -->
+            <param name="gravity_comp_L1_sin">0.0</param>
+            <param name="gravity_comp_L1_cos">0.0</param>
+            <param name="gravity_comp_L1_offset">0.0</param>
+            <!-- L2 joint - Upper arm pitch, bears primary gravity load -->
+            <!-- tau = m*g*L*sin(theta), needs calibration based on actual measurements -->
+            <param name="gravity_comp_L2_sin">3.5</param>
+            <param name="gravity_comp_L2_cos">0.0</param>
+            <param name="gravity_comp_L2_offset">0.0</param>
+            <!-- L3 joint - Forearm pitch -->
+            <param name="gravity_comp_L3_sin">2.0</param>
+            <param name="gravity_comp_L3_cos">0.0</param>
+            <param name="gravity_comp_L3_offset">0.0</param>
+            <!-- L4 joint - Wrist Roll -->
+            <param name="gravity_comp_L4_sin">0.0</param>
+            <param name="gravity_comp_L4_cos">0.0</param>
+            <param name="gravity_comp_L4_offset">0.0</param>
+            <!-- L5 joint - Wrist Pitch -->
+            <param name="gravity_comp_L5_sin">0.3</param>
+            <param name="gravity_comp_L5_cos">0.0</param>
+            <param name="gravity_comp_L5_offset">0.0</param>
+            <!-- L6 joint - Wrist Yaw -->
+            <param name="gravity_comp_L6_sin">0.0</param>
+            <param name="gravity_comp_L6_cos">0.0</param>
+            <param name="gravity_comp_L6_offset">0.0</param>
+          </xacro:unless>
         </xacro:unless>
       </hardware>
